File: hardware/p1s.brd (EAGLE design)
At the start: 95 x 72 mm, 32 parts, among them IC1 74LS595N, IC2 74ALS04N, IC3 74ALS04N, J0 DC24V, Q1 60V/32A/35mΩ, Q2 60V/32A/35mΩ, Q3 60V/32A/35mΩ, Q4 60V/32A/35mΩ, Q5 60V/32A/35mΩ, Q6 60V/32A/35mΩ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

Commit message: Updated P1S.
Parts:
- removed J1, J2: (no value), SparkFun-Connectors:JST-5-PTH
- added SV2: (no value), con-ml:ML10L
- added SV3: (no value), con-ml:ML16L
- SV1: device con-ml:ML16L -> con-ml:ML10L
- moved SV1 44.2 mm to (11.0, 36.0), turned to 90 degrees
- moved R1 34.1 mm to (31.0, 24.0)
- moved J0 12.0 mm to (81.0, 61.0)
- moved R2 5.10 mm to (64.0, 24.0)
- moved D1 5.00 mm to (21.0, 47.0)
- moved Q1 5.00 mm to (21.0, 51.0)
- moved D2 4.00 mm to (20.0, 33.0)
- moved D3 4.00 mm to (20.0, 19.0)
- moved D4 4.00 mm to (20.0, 5.00)
- moved D5 4.00 mm to (75.0, 47.0)
- moved D6 4.00 mm to (75.0, 33.0)
- moved D7 4.00 mm to (75.0, 19.0)
- moved D8 4.00 mm to (75.0, 5.00)
- moved Q2 4.00 mm to (20.0, 37.0)
- moved Q3 4.00 mm to (20.0, 23.0)
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Connections:
- new net IC1: SV1.9, SV2.9
- new net IC2: SV1.10, SV2.10
- net +24V: now also SV3.1, SV3.11, SV3.13, SV3.15, SV3.3, SV3.5, SV3.7, SV3.9; no longer SV1.1, SV1.11, SV1.13, SV1.15, SV1.3, SV1.5, SV1.7, SV1.9
- net GND: now also SV1.2, SV2.2; no longer J1.2, J2.2
- net RCLK: now also SV1.3, SV2.3; no longer J1.3, J2.3
- net SCLK: now also SV1.4, SV2.4; no longer J1.4, J2.4
- net SIN: now also SV1.5; no longer J1.5
- net SOUT: now also SV2.5; no longer J2.5
- net VCC: now also SV1.1, SV2.1; no longer J1.1, J2.1
- net X1: now also SV3.2; no longer SV1.2
- net X2: now also SV3.4; no longer SV1.4
- net X3: now also SV3.6; no longer SV1.6
- net X4: now also SV3.8; no longer SV1.8
- net X5: now also SV3.10; no longer SV1.10
- net X6: now also SV3.12; no longer SV1.12
- net X7: now also SV3.14; no longer SV1.14
- net X8: now also SV3.16; no longer SV1.16
Routing:
- net IC2: track 0.00 -> 124.7 mm
- net IC1: track 0.00 -> 102.5 mm, vias 0 -> 1
- net N$1: track 87.8 -> 122.6 mm
- net D3: track 95.4 -> 66.6 mm
- net N$4: track 63.0 -> 85.5 mm
- net X2: track 61.7 -> 41.2 mm, vias 0 -> 1
- net D5: track 57.2 -> 74.8 mm, vias 0 -> 1
- net +24V: track 159.1 -> 176.6 mm, vias 4 -> 3
- net D7: track 95.3 -> 112.8 mm
- net SCLK: track 169.7 -> 153.4 mm
- net N$25: track 26.4 -> 13.6 mm
- net N$12: track 62.0 -> 50.1 mm, vias 0 -> 1
- net SOUT: track 83.7 -> 72.7 mm
- net X7: track 70.2 -> 60.3 mm
- net D4: track 58.8 -> 68.3 mm
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