File: hardware/catbit.brd (EAGLE design)
At the start: 95 x 72 mm, 37 parts, among them J0 DC24V, Q1 60V/32A/35mΩ, Q2 60V/32A/35mΩ, Q3 60V/32A/35mΩ, Q4 60V/32A/35mΩ, Q5 60V/32A/35mΩ, Q6 60V/32A/35mΩ, Q7 60V/32A/35mΩ, Q8 60V/32A/35mΩ

Commit message: Removed capacitance value.
Parts:
- C1, C2: value 0.01u -> (none)
Changed lines of the file:
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@@
 <attribute name="VALUE" x="1.475" y="14.365" size="0.889" layer="27" ratio="11"/>
 </element>
-<element name="C1" library="resistor" library_urn="urn:adsk.eagle:library:348" package="C025-024X044" package3d_urn="urn:adsk.eagle:package:26149/1" value="0.01u" x="20" y="12" smashed="yes" rot="R90">
+<element name="C1" library="resistor" library_urn="urn:adsk.eagle:library:348" package="C025-024X044" package3d_urn="urn:adsk.eagle:package:26149/1" value="" x="20" y="12" smashed="yes" rot="R90">
 <attribute name="NAME" x="20" y="14.5" size="1" layer="25" ratio="10" align="bottom-center"/>
 <attribute name="VALUE" x="22.667" y="10.222" size="1.27" layer="27" ratio="10" rot="R90"/>
 </element>
-<element name="C2" library="resistor" library_urn="urn:adsk.eagle:library:348" package="C025-024X044" package3d_urn="urn:adsk.eagle:package:26149/1" value="0.01u" x="28" y="12" smashed="yes" rot="R90">
+<element name="C2" library="resistor" library_urn="urn:adsk.eagle:library:348" package="C025-024X044" package3d_urn="urn:adsk.eagle:package:26149/1" value="" x="28" y="12" smashed="yes" rot="R90">
 <attribute name="NAME" x="28" y="9.5" size="1" layer="25" ratio="10" rot="R180" align="bottom-center"/>
 <attribute name="VALUE" x="30.667" y="10.222" size="1.27" layer="27" ratio="10" rot="R90"/>

Commit message: Design of the board.
Parts:
- moved LOGO1 76.0 mm to (86.0, 5.00)
- moved U$1 40.3 mm to (47.5, 66.0)
- moved OK5 14.0 mm to (61.0, 62.0)
- moved OK7 14.0 mm to (61.0, 36.0)
- moved OK8 14.0 mm to (61.0, 23.0)
- moved OK6 14.0 mm to (61.0, 49.0)
- moved Q5 13.2 mm to (76.0, 62.0), turned to 270 degrees
- moved Q6 13.0 mm to (76.0, 49.0), turned to 270 degrees
- moved Q7 13.0 mm to (76.0, 36.0), turned to 270 degrees
- moved Q8 13.0 mm to (76.0, 23.0), turned to 270 degrees
- moved D7 9.85 mm to (72.0, 36.0), turned to 90 degrees
- moved D8 9.85 mm to (72.0, 23.0), turned to 90 degrees
- moved D6 9.49 mm to (72.0, 49.0), turned to 90 degrees
- moved D5 9.22 mm to (72.0, 62.0), turned to 90 degrees
- moved RN2 6.00 mm to (47.5, 51.0)
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Routing:
- net GNDA: track 170.7 -> 213.1 mm, vias 1 -> 2
- net +24V: track 178.8 -> 215.6 mm, vias 0 -> 1
- net VCC: track 181.3 -> 148.8 mm, vias 0 -> 3
- net X7: track 71.0 -> 101.2 mm
- net X8: track 80.7 -> 109.9 mm
- net X5: track 74.0 -> 101.8 mm
- net X6: track 73.4 -> 99.1 mm
- net GND: track 217.9 -> 238.2 mm, vias 1 -> 3
- net D3: track 79.6 -> 99.5 mm
- net N$9: track 70.5 -> 50.5 mm
- net N$1: track 90.3 -> 108.6 mm, vias 2 -> 1
- net N$6: track 71.6 -> 54.7 mm
- net N$23: track 44.3 -> 27.6 mm
- net D1: track 118.6 -> 102.2 mm
- net N$20: track 37.5 -> 21.4 mm
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- added copper zone on layer 1, net GND
- added copper zone on layer 16, net GND
Other:
- board text added: "1"
- board text added: "CatBit-8 1.0.0-X"
- board text added: "Common V+"
- board text added: "Digital Input x8"
- board text added: "Power Output x8"
- board text removed: "Cat-8 1.0.0-X"
