File: hardware/catbit.sch (EAGLE design)
At the start: 37 parts, among them J0 DC24V, Q1 60V/32A/35mΩ, Q2 60V/32A/35mΩ, Q3 60V/32A/35mΩ, Q4 60V/32A/35mΩ, Q5 60V/32A/35mΩ, Q6 60V/32A/35mΩ, Q7 60V/32A/35mΩ, Q8 60V/32A/35mΩ

Commit message: Removed capacitance value.
Parts:
- C1, C2: value 0.01u -> (none)
Changed lines of the file:
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@@
 <part name="J0" library="Seeed-Connector" library_urn="urn:adsk.eagle:library:478" deviceset="JACK-DC-005" device="'DC-005'" package3d_urn="urn:adsk.eagle:package:33150/1" value="DC24V"/>
 <part name="FRAME1" library="frames" library_urn="urn:adsk.eagle:library:229" deviceset="A4L-LOC" device=""/>
-<part name="C1" library="resistor" library_urn="urn:adsk.eagle:library:348" deviceset="C-EU" device="025-024X044" package3d_urn="urn:adsk.eagle:package:26149/1" value="0.01u"/>
-<part name="C2" library="resistor" library_urn="urn:adsk.eagle:library:348" deviceset="C-EU" device="025-024X044" package3d_urn="urn:adsk.eagle:package:26149/1" value="0.01u"/>
+<part name="C1" library="resistor" library_urn="urn:adsk.eagle:library:348" deviceset="C-EU" device="025-024X044" package3d_urn="urn:adsk.eagle:package:26149/1"/>
+<part name="C2" library="resistor" library_urn="urn:adsk.eagle:library:348" deviceset="C-EU" device="025-024X044" package3d_urn="urn:adsk.eagle:package:26149/1"/>
 <part name="SUPPLY1" library="supply2" deviceset="GND" device=""/>
 <part name="P+1" library="supply1" library_urn="urn:adsk.eagle:library:371" deviceset="+24V" device=""/>

Commit message: Renamed DZ1 to L1.
Parts:
- renumbered DZ1 to L1
Changed lines of the file:
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@@
 <part name="OK1" library="optocoupler" library_urn="urn:adsk.eagle:library:320" deviceset="6N137" device="" package3d_urn="urn:adsk.eagle:package:21941/1"/>
 <part name="RN1" library="resistor-dil" library_urn="urn:adsk.eagle:library:342" deviceset="8R-N" device="" package3d_urn="urn:adsk.eagle:package:922/2"/>
-<part name="DZ1" library="led" library_urn="urn:adsk.eagle:library:259" deviceset="LB10" device="" package3d_urn="urn:adsk.eagle:package:15791/1"/>
+<part name="L1" library="led" library_urn="urn:adsk.eagle:library:259" deviceset="LB10" device="" package3d_urn="urn:adsk.eagle:package:15791/1"/>
 <part name="SUPPLY4" library="supply2" deviceset="GND" device=""/>
 <part name="P+4" library="supply1" library_urn="urn:adsk.eagle:library:371" deviceset="VCC" device=""/>
@@
 <attribute name="NAME" x="109.22" y="32.512" size="1.778" layer="95"/>
 </instance>
-<instance part="DZ1" gate="-1" x="20.32" y="144.78" smashed="yes">
+<instance part="L1" gate="-1" x="20.32" y="144.78" smashed="yes">
 <attribute name="NAME" x="23.876" y="140.462" size="1.778" layer="95" rot="R90"/>
 <attribute name="VALUE" x="26.035" y="140.462" size="1.778" layer="96" rot="R90"/>
 </instance>
-<instance part="DZ1" gate="-2" x="20.32" y="106.68" smashed="yes">
+<instance part="L1" gate="-2" x="20.32" y="106.68" smashed="yes">
 <attribute name="NAME" x="23.876" y="102.362" size="1.778" layer="95" rot="R90"/>
 <attribute name="VALUE" x="26.035" y="102.362" size="1.778" layer="96" rot="R90"/>
 </instance>
-<instance part="DZ1" gate="-3" x="20.32" y="68.58" smashed="yes">
+<instance part="L1" gate="-3" x="20.32" y="68.58" smashed="yes">
 <attribute name="NAME" x="23.876" y="64.262" size="1.778" layer="95" rot="R90"/>
 <attribute name="VALUE" x="26.035" y="64.262" size="1.778" layer="96" rot="R90"/>
 </instance>
-<instance part="DZ1" gate="-4" x="20.32" y="30.48" smashed="yes">
+<instance part="L1" gate="-4" x="20.32" y="30.48" smashed="yes">
 <attribute name="NAME" x="23.876" y="26.162" size="1.778" layer="95" rot="R90"/>
 <attribute name="VALUE" x="26.035" y="26.162" size="1.778" layer="96" rot="R90"/>
 </instance>
-<instance part="DZ1" gate="-5" x="121.92" y="144.78" smashed="yes">
+<instance part="L1" gate="-5" x="121.92" y="144.78" smashed="yes">
 <attribute name="NAME" x="125.476" y="140.462" size="1.778" layer="95" rot="R90"/>
 <attribute name="VALUE" x="127.635" y="140.462" size="1.778" layer="96" rot="R90"/>
 </instance>
-<instance part="DZ1" gate="-6" x="121.92" y="106.68" smashed="yes">
+<instance part="L1" gate="-6" x="121.92" y="106.68" smashed="yes">
 <attribute name="NAME" x="125.476" y="102.362" size="1.778" layer="95" rot="R90"/>
 <attribute name="VALUE" x="127.635" y="102.362" size="1.778" layer="96" rot="R90"/>
 </instance>
-<instance part="DZ1" gate="-7" x="121.92" y="68.58" smashed="yes">
+<instance part="L1" gate="-7" x="121.92" y="68.58" smashed="yes">
 <attribute name="NAME" x="125.476" y="64.262" size="1.778" layer="95" rot="R90"/>
 <attribute name="VALUE" x="127.635" y="64.262" size="1.778" layer="96" rot="R90"/>
 </instance>
-<instance part="DZ1" gate="-8" x="121.92" y="30.48" smashed="yes">
+<instance part="L1" gate="-8" x="121.92" y="30.48" smashed="yes">
 <attribute name="NAME" x="125.476" y="26.162" size="1.778" layer="95" rot="R90"/>
 <attribute name="VALUE" x="127.635" y="26.162" size="1.778" layer="96" rot="R90"/>
 </instance>
-<instance part="DZ1" gate="-9" x="132.08" y="7.62" smashed="yes">
+<instance part="L1" gate="-9" x="132.08" y="7.62" smashed="yes">
 <attribute name="NAME" x="135.636" y="3.302" size="1.778" layer="95" rot="R90"/>
 <attribute name="VALUE" x="137.795" y="3.302" size="1.778" layer="96" rot="R90"/>
 </instance>
-<instance part="DZ1" gate="-10" x="142.24" y="7.62" smashed="yes">
+<instance part="L1" gate="-10" x="142.24" y="7.62" smashed="yes">
 <attribute name="NAME" x="145.796" y="3.302" size="1.778" layer="95" rot="R90"/>
 <attribute name="VALUE" x="147.955" y="3.302" size="1.778" layer="96" rot="R90"/>
@@
 </segment>
 <segment>
-<pinref part="DZ1" gate="-1" pin="C"/>
+<pinref part="L1" gate="-1" pin="C"/>
 <wire x1="20.32" y1="139.7" x2="20.32" y2="137.16" width="0.1524" layer="91"/>
 <pinref part="SUPPLY12" gate="GND" pin="GND"/>
 </segment>
 <segment>
-<pinref part="DZ1" gate="-2" pin="C"/>
+<pinref part="L1" gate="-2" pin="C"/>
 <pinref part="SUPPLY14" gate="GND" pin="GND"/>
 <wire x1="20.32" y1="99.06" x2="20.32" y2="101.6" width="0.1524" layer="91"/>
 </segment>
 <segment>
-<pinref part="DZ1" gate="-3" pin="C"/>
+<pinref part="L1" gate="-3" pin="C"/>
 <pinref part="SUPPLY15" gate="GND" pin="GND"/>
 <wire x1="20.32" y1="60.96" x2="20.32" y2="63.5" width="0.1524" layer="91"/>
 </segment>
 <segment>
-<pinref part="DZ1" gate="-4" pin="C"/>
+<pinref part="L1" gate="-4" pin="C"/>
 <pinref part="SUPPLY16" gate="GND" pin="GND"/>
 <wire x1="20.32" y1="22.86" x2="20.32" y2="25.4" width="0.1524" layer="91"/>
 </segment>
 <segment>
-<pinref part="DZ1" gate="-8" pin="C"/>
+<pinref part="L1" gate="-8" pin="C"/>
 <pinref part="SUPPLY17" gate="GND" pin="GND"/>
 <wire x1="121.92" y1="22.86" x2="121.92" y2="25.4" width="0.1524" layer="91"/>
 </segment>
 <segment>
-<pinref part="DZ1" gate="-7" pin="C"/>
+<pinref part="L1" gate="-7" pin="C"/>
 <pinref part="SUPPLY18" gate="GND" pin="GND"/>
 <wire x1="121.92" y1="60.96" x2="121.92" y2="63.5" width="0.1524" layer="91"/>
 </segment>
 <segment>
-<pinref part="DZ1" gate="-6" pin="C"/>
+<pinref part="L1" gate="-6" pin="C"/>
 <pinref part="SUPPLY19" gate="GND" pin="GND"/>
 <wire x1="121.92" y1="99.06" x2="121.92" y2="101.6" width="0.1524" layer="91"/>
 </segment>
 <segment>
-<pinref part="DZ1" gate="-5" pin="C"/>
+<pinref part="L1" gate="-5" pin="C"/>
 <pinref part="SUPPLY13" gate="GND" pin="GND"/>
 <wire x1="121.92" y1="137.16" x2="121.92" y2="139.7" width="0.1524" layer="91"/>
@@
 <wire x1="25.4" y1="149.86" x2="20.32" y2="149.86" width="0.1524" layer="91"/>
 <pinref part="RN1" gate="A" pin="2"/>
-<pinref part="DZ1" gate="-1" pin="A"/>
+<pinref part="L1" gate="-1" pin="A"/>
 <wire x1="20.32" y1="149.86" x2="17.78" y2="149.86" width="0.1524" layer="91"/>
 <wire x1="20.32" y1="149.86" x2="20.32" y2="147.32" width="0.1524" layer="91"/>
@@
 <wire x1="25.4" y1="111.76" x2="20.32" y2="111.76" width="0.1524" layer="91"/>
 <pinref part="RN1" gate="B" pin="2"/>
-<pinref part="DZ1" gate="-2" pin="A"/>
+<pinref part="L1" gate="-2" pin="A"/>
 <wire x1="20.32" y1="111.76" x2="17.78" y2="111.76" width="0.1524" layer="91"/>
 <wire x1="20.32" y1="111.76" x2="20.32" y2="109.22" width="0.1524" layer="91"/>
@@
 <wire x1="25.4" y1="73.66" x2="20.32" y2="73.66" width="0.1524" layer="91"/>
 <pinref part="RN1" gate="C" pin="2"/>
-<pinref part="DZ1" gate="-3" pin="A"/>
+<pinref part="L1" gate="-3" pin="A"/>
 <wire x1="20.32" y1="73.66" x2="17.78" y2="73.66" width="0.1524" layer="91"/>
 <wire x1="20.32" y1="73.66" x2="20.32" y2="71.12" width="0.1524" layer="91"/>
@@
 <wire x1="25.4" y1="35.56" x2="20.32" y2="35.56" width="0.1524" layer="91"/>
 <pinref part="RN1" gate="D" pin="2"/>
-<pinref part="DZ1" gate="-4" pin="A"/>
+<pinref part="L1" gate="-4" pin="A"/>
 <wire x1="20.32" y1="35.56" x2="17.78" y2="35.56" width="0.1524" layer="91"/>
 <wire x1="20.32" y1="35.56" x2="20.32" y2="33.02" width="0.1524" layer="91"/>
@@
 <wire x1="127" y1="149.86" x2="121.92" y2="149.86" width="0.1524" layer="91"/>
 <pinref part="RN1" gate="E" pin="2"/>
-<pinref part="DZ1" gate="-5" pin="A"/>
+<pinref part="L1" gate="-5" pin="A"/>
 <wire x1="121.92" y1="149.86" x2="119.38" y2="149.86" width="0.1524" layer="91"/>
 <wire x1="121.92" y1="149.86" x2="121.92" y2="147.32" width="0.1524" layer="91"/>
@@
 <wire x1="127" y1="111.76" x2="121.92" y2="111.76" width="0.1524" layer="91"/>
 <pinref part="RN1" gate="F" pin="2"/>
-<pinref part="DZ1" gate="-6" pin="A"/>
+<pinref part="L1" gate="-6" pin="A"/>
 <wire x1="121.92" y1="111.76" x2="119.38" y2="111.76" width="0.1524" layer="91"/>
 <wire x1="121.92" y1="111.76" x2="121.92" y2="109.22" width="0.1524" layer="91"/>
@@
 <wire x1="127" y1="73.66" x2="121.92" y2="73.66" width="0.1524" layer="91"/>
 <pinref part="RN1" gate="G" pin="2"/>
-<pinref part="DZ1" gate="-7" pin="A"/>
+<pinref part="L1" gate="-7" pin="A"/>
 <wire x1="121.92" y1="73.66" x2="119.38" y2="73.66" width="0.1524" layer="91"/>
 <wire x1="121.92" y1="73.66" x2="121.92" y2="71.12" width="0.1524" layer="91"/>
@@
 <wire x1="127" y1="35.56" x2="121.92" y2="35.56" width="0.1524" layer="91"/>
 <pinref part="RN1" gate="H" pin="2"/>
-<pinref part="DZ1" gate="-8" pin="A"/>
+<pinref part="L1" gate="-8" pin="A"/>
 <wire x1="121.92" y1="35.56" x2="119.38" y2="35.56" width="0.1524" layer="91"/>
 <wire x1="121.92" y1="35.56" x2="121.92" y2="33.02" width="0.1524" layer="91"/>

Commit message: Fixed GND separation.
Connections:
- net GND: no longer C1.2, C2.2, IC1.GND, OK1.GND, OK2.GND, OK3.GND, OK4.GND, OK5.GND, OK6.GND, OK7.GND, OK8.GND
- net GNDA: now also C1.2, C2.2, IC1.GND, OK1.GND, OK2.GND, OK3.GND, OK4.GND, OK5.GND, OK6.GND, OK7.GND, OK8.GND

Commit message: Silk.
Parts:
- RN1: value (none) -> 160
- RN2: value (none) -> 100
- RN3: value (none) -> 1k
Changed lines of the file:
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@@
 <part name="SUPPLY3" library="supply2" deviceset="GND" device=""/>
 <part name="OK1" library="optocoupler" library_urn="urn:adsk.eagle:library:320" deviceset="6N137" device="" package3d_urn="urn:adsk.eagle:package:21941/1"/>
-<part name="RN1" library="resistor-dil" library_urn="urn:adsk.eagle:library:342" deviceset="8R-N" device="" package3d_urn="urn:adsk.eagle:package:922/2"/>
+<part name="RN1" library="resistor-dil" library_urn="urn:adsk.eagle:library:342" deviceset="8R-N" device="" package3d_urn="urn:adsk.eagle:package:922/2" value="160"/>
 <part name="L1" library="led" library_urn="urn:adsk.eagle:library:259" deviceset="LB10" device="" package3d_urn="urn:adsk.eagle:package:15791/1"/>
 <part name="SUPPLY4" library="supply2" deviceset="GND" device=""/>
 <part name="P+4" library="supply1" library_urn="urn:adsk.eagle:library:371" deviceset="VCC" device=""/>
-<part name="RN2" library="resistor-dil" library_urn="urn:adsk.eagle:library:342" deviceset="8R-N" device="" package3d_urn="urn:adsk.eagle:package:922/2"/>
-<part name="RN3" library="resistor-dil" library_urn="urn:adsk.eagle:library:342" deviceset="8R-N" device="" package3d_urn="urn:adsk.eagle:package:922/2"/>
+<part name="RN2" library="resistor-dil" library_urn="urn:adsk.eagle:library:342" deviceset="8R-N" device="" package3d_urn="urn:adsk.eagle:package:922/2" value="100"/>
+<part name="RN3" library="resistor-dil" library_urn="urn:adsk.eagle:library:342" deviceset="8R-N" device="" package3d_urn="urn:adsk.eagle:package:922/2" value="1k"/>
 <part name="GND2" library="supply1" library_urn="urn:adsk.eagle:library:371" deviceset="GNDA" device=""/>
 <part name="Q1" library="SparkFun-DiscreteSemi" library_urn="urn:adsk.eagle:library:514" deviceset="MOSFET-NCH" device="-FQP30N06L" package3d_urn="urn:adsk.eagle:package:38447/1" value="60V/32A/35mΩ"/>
